File: Rapid Training Target/Rapid Training Target.kicad_sch (KiCad schematic)
At the start: 1 part

Commit message: First revision of the PCB
Parts:
- removed U1: ~, Personal:QFN33P50_500X500X90L40X25T370N, symbol personal2:ESP32_C3
- added D1, D2, D3, D4, D5: LED_ARBG, Personal:DIODFN4_100X100X35L29X29N, symbol Device:LED_ARBG
- added H1, H2, H3: MountingHole, MountingHole:MountingHole_3.2mm_M3_DIN965_Pad, symbol Mechanical:MountingHole
- added Q1, Q2, Q3: 2N7002, Package_TO_SOT_SMD:SOT-23, symbol Transistor_FET:2N7002
- added R10: 2.7k, Resistor_SMD:R_0603_1608Metric, symbol Device:R
- added R11: 5.6k, Resistor_SMD:R_0603_1608Metric, symbol Device:R
- added R12: 1.5k, Resistor_SMD:R_0603_1608Metric, symbol Device:R
- added U1: ~, Personal:ESP32-C3-DevKit, symbol personal2:ESP32-C3_DevKit_Rev_A
Connections:
- net +3V3: now also U1.18 (3V3)
- net GND: now also Q1.3 (D), Q2.3 (D), Q3.3 (D), U1.17 (GND), U1.2 (GND)
- new net: D1.2 (RK), D2.2 (RK), D3.2 (RK), D4.2 (RK), D5.2 (RK), R10.1
- new net: D1.3 (BK), D2.3 (BK), D3.3 (BK), D4.3 (BK), D5.3 (BK), R12.1
- new net: D1.4 (GK), D2.4 (GK), D3.4 (GK), D4.4 (GK), D5.4 (GK), R11.1
- new net: Q2.2 (S), R11.2
- new net: Q1.2 (S), R10.2
- new net: Q3.2 (S), R12.2
- new net +5V: D1.1 (A), D2.1 (A), D3.1 (A), D4.1 (A), D5.1 (A), U1.1 (5V)
- new net Blue: Q3.1 (G), U1.9 (GPIO6)
- new net Green: Q2.1 (G), U1.8 (GPIO5)
- new net Red: Q1.1 (G), U1.7 (GPIO4)
