File: Hardware/Rapid Training Target/Rapid Training Target.kicad_sch (KiCad schematic)
At the start: 17 parts, among them U1 MIC5504-3.3YM5, U2 ESP32-C3-MINI-1-N4

Commit message: added a boot bridge jumper
Parts:
- added JP1: SolderJumper_2_Bridged, Jumper:SolderJumper-2_P1.3mm_Bridged_RoundedPad1.0x1.5mm, symbol Jumper:SolderJumper_2_Bridged
Connections:
- net GND: now also JP1.2 (B)
- net at U2.23 (IO9/GPIO9): now also JP1.1 (A)
Changed lines of the file:
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@@
+    (stroke (width 0) (type default))
+  )
+  (wire (pts (xy 231.14 90.17) (xy 232.41 90.17))
     (stroke (width 0) (type default))
   )
@@
     (stroke (width 0) (type default))
   )
+  (wire (pts (xy 212.09 90.17) (xy 223.52 90.17))
+    (stroke (width 0) (type default))
+  )
   (wire (pts (xy 29.21 143.51) (xy 30.48 143.51))
     (stroke (width 0) (type default))
@@
   )
   (wire (pts (xy 29.21 158.75) (xy 38.1 158.75))
+    (stroke (width 0) (type default))
+  )
+  (wire (pts (xy 232.41 90.17) (xy 232.41 91.44))
     (stroke (width 0) (type default))
   )
@@
     )
   )
+  (symbol (lib_id "Jumper:SolderJumper_2_Bridged") (at 227.33 90.17 0) (unit 1)
+    (in_bom yes) (on_board yes) (dnp no) (fields_autoplaced)
+    (property "Reference" "JP1" (at 227.33 83.82 0)
+      (effects (font (size 1.27 1.27)))
+    )
+    (property "Value" "SolderJumper_2_Bridged" (at 227.33 86.36 0)
+      (effects (font (size 1.27 1.27)))
+    )
+    (property "Footprint" "Jumper:SolderJumper-2_P1.3mm_Bridged_RoundedPad1.0x1.5mm" (at 227.33 90.17 0)
+      (effects (font (size 1.27 1.27)) hide)
+    )
+    (property "Datasheet" "~" (at 227.33 90.17 0)
+      (effects (font (size 1.27 1.27)) hide)
+    )
+    (pin "1")
+    (pin "2")
+    (instances
+      (project "Rapid Training Target"
+        (path "/9fedd953-8356-4168-99e6-03d50e1e6951"
+          (reference "JP1") (unit 1)
+        )
+      )
+    )
+  )
+  (symbol (lib_name "GND_4") (lib_id "power:GND") (at 232.41 91.44 0) (unit 1)
+    (in_bom yes) (on_board yes) (dnp no) (fields_autoplaced)
+    (property "Reference" "#PWR03" (at 232.41 97.79 0)
+      (effects (font (size 1.27 1.27)) hide)
+    )
+    (property "Value" "GND" (at 232.41 96.52 0)
+      (effects (font (size 1.27 1.27)))
+    )
+    (property "Footprint" "" (at 232.41 91.44 0)
+      (effects (font (size 1.27 1.27)) hide)
+    )
+    (property "Datasheet" "" (at 232.41 91.44 0)
+      (effects (font (size 1.27 1.27)) hide)
+    )
+    (pin "1")
+    (instances
+      (project "Rapid Training Target"
+        (path "/9fedd953-8356-4168-99e6-03d50e1e6951"
+          (reference "#PWR03") (unit 1)
+        )
+      )
+    )
+  )

Commit message: added bom and pos files
Parts:
- JP1: footprint Jumper:SolderJumper-2_P1.3mm_Bridged_RoundedPad1.0x1.5mm -> Jumper:SolderJumper-2_P1.3mm_Open_RoundedPad1.0x1.5mm; symbol Jumper:SolderJumper_2_Bridged -> Jumper:SolderJumper_2_Open
Connections:
- net +3V3: now also U2.22 (IO8/GPIO8), U2.5 (IO2/GPIO2/ADC1_CH2/FSPIQ)
Other:
- company: (none) -> Rev C: Added Bootstrapping
Changed lines of the file:
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@@
   (title_block
     (title "Rapid Training Target")
-    (date "2023-06-27")
-    (rev "B")
+    (date "2023-08-28")
+    (rev "C")
+    (company "Rev C: Added Bootstrapping")
     (comment 1 "Rev B: Change to integrated MCU")
     (comment 2 "Rev A: Initial Commit")
@@
   (junction (at 149.86 135.89) (diameter 0) (color 0 0 0 0)
   )
+  (junction (at 213.36 72.39) (diameter 0) (color 0 0 0 0)
+  )
   (junction (at 93.98 41.91) (diameter 0) (color 0 0 0 0)
   )
@@
   (junction (at 35.56 179.07) (diameter 0) (color 0 0 0 0)
   )
+  (wire (pts (xy 213.36 87.63) (xy 213.36 72.39))
+    (stroke (width 0) (type default))
+  )
   (wire (pts (xy 35.56 179.07) (xy 35.56 176.53))
     (stroke (width 0) (type default))
@@
     (stroke (width 0) (type default))
   )
+  (wire (pts (xy 213.36 66.04) (xy 213.36 72.39))
+    (stroke (width 0) (type default))
+  )
   (wire (pts (xy 149.86 87.63) (xy 149.86 90.17))
     (stroke (width 0) (type default))
@@
     (stroke (width 0) (type default))
   )
+  (wire (pts (xy 212.09 87.63) (xy 213.36 87.63))
+    (stroke (width 0) (type default))
+  )
   (wire (pts (xy 149.86 100.33) (xy 149.86 102.87))
     (stroke (width 0) (type default))
@@
   )
   (wire (pts (xy 35.56 49.53) (xy 88.9 49.53))
+    (stroke (width 0) (type default))
+  )
+  (wire (pts (xy 213.36 72.39) (xy 212.09 72.39))
     (stroke (width 0) (type default))
   )
@@
     )
   )
-  (symbol (lib_id "Jumper:SolderJumper_2_Bridged") (at 227.33 90.17 0) (unit 1)
+  (symbol (lib_id "Jumper:SolderJumper_2_Open") (at 227.33 90.17 0) (unit 1)
     (in_bom yes) (on_board yes) (dnp no) (fields_autoplaced)
     (property "Reference" "JP1" (at 227.33 83.82 0)
@@
       (effects (font (size 1.27 1.27)))
     )
-    (property "Footprint" "Jumper:SolderJumper-2_P1.3mm_Bridged_RoundedPad1.0x1.5mm" (at 227.33 90.17 0)
+    (property "Footprint" "Jumper:SolderJumper-2_P1.3mm_Open_RoundedPad1.0x1.5mm" (at 227.33 90.17 0)
       (effects (font (size 1.27 1.27)) hide)
     )
@@
         )
       )
+    )
+  )
+  (symbol (lib_id "power:+3V3") (at 213.36 66.04 0) (unit 1)
+    (in_bom yes) (on_board yes) (dnp no) (fields_autoplaced)
+    (property "Reference" "#PWR04" (at 213.36 69.85 0)
+      (effects (font (size 1.27 1.27)) hide)
+    )
+    (property "Value" "+3V3" (at 213.36 60.96 0)
+      (effects (font (size 1.27 1.27)))
+    )
+    (property "Footprint" "" (at 213.36 66.04 0)
+      (effects (font (size 1.27 1.27)) hide)
+    )
+    (property "Datasheet" "" (at 213.36 66.04 0)
+      (effects (font (size 1.27 1.27)) hide)
+    )
+    (pin "1")
+    (instances
+      (project "Rapid Training Target"
+        (path "/9fedd953-8356-4168-99e6-03d50e1e6951"
+          (reference "#PWR04") (unit 1)
+        )
+      )
