File: Hardware/Rapid Training Target/Rapid_Training_Target.kicad_sch (KiCad schematic)
At the start: 23 parts, among them U1 MIC5504-3.3YM5, U3 ESP32-C3-MINI-1

Commit message: Updated Footprints for LED
Parts:
- D1, D2, D3, D4, D5: footprint Personal:DIODFN4_100X100X35L29X29N -> training:DIODFN4_100X100X35L29X29N
